File: getting-started.kicad_sch (KiCad schematic)
At the start: 4 parts, among them SW1 M2011S3A1W03

Commit message: propogating changes through sch and bom
Parts:
- SW1: footprint getting-started:Untitled -> getting-started:M2011S3A1W03
Changed lines of the file:
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@@
 			)
 		)
-		(property "Footprint" "getting-started:Untitled"
+		(property "Footprint" "getting-started:M2011S3A1W03"
 			(at 115.57 89.916 0)
 			(effects
