File: getting-started.kicad_pcb (KiCad board)
At the start: 2 copper layers, 49 x 34 mm, 4 parts, among them SW1 M2011S3A1W03

Commit message: propogating changes through pcb
Parts:
- SW1: footprint getting-started:Untitled -> getting-started:M2011S3A1W03
Changed lines of the file:
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@@
 		)
 	)
-	(footprint "getting-started:Untitled"
+	(footprint "getting-started:M2011S3A1W03"
 		(layer "F.Cu")
 		(at 156 89.6)
